Commit message: Added rviz and gazebo launch files

File: src/diff_drive_robot/urdf/diff_drive_robot.xacro (robot description, xacro)
@@ -119,5 +119,5 @@
     <child link="left_wheel_link"/>
     <!-- Wheel center -->
-    <origin xyz="0 ${s/2} ${wheel_radius}"
+    <origin xyz="0 ${s/2} ${wheel_radius/2}"
             rpy="0 0 0"/>
     <!-- Wheel rotates around Y -->
@@ -132,5 +132,5 @@
     <child link="right_wheel_link"/>
     <!-- Wheel center -->
-    <origin xyz="0 -${s/2} ${wheel_radius}"
+    <origin xyz="0 -${s/2} ${wheel_radius/2}"
             rpy="0 0 0"/>
     <!-- Wheel rotates around Y -->

Commit message: Added caster wheel and tested the moving dynamics and the plugin

File: src/diff_drive_robot/urdf/diff_drive_robot.xacro (robot description, xacro)
@@ -15,4 +15,12 @@
   <xacro:property name="wheel_radius" value="0.10"/>
   <xacro:property name="wheel_width"  value="0.05"/>
+  <!-- Low-friction fixed front support sphere -->
+  <xacro:property name="caster_sphere_radius" value="0.05"/>
+  <xacro:property name="caster_sphere_mass" value="0.20"/>
+  <xacro:property name="caster_sphere_x"
+                  value="0.22"/>
+  <!-- Sphere bottom matches the drive wheels' contact height. -->
+  <xacro:property name="caster_sphere_z"
+                  value="${wheel_radius / 2 - caster_sphere_radius}"/>
   <!-- Masses -->
   <xacro:property name="body_mass"  value="5.0"/>
@@ -112,4 +120,31 @@
   </link>
   <!-- ========================================================= -->
+  <!-- Fixed Low-Friction Front Sphere                           -->
+  <!-- ========================================================= -->
+  <link name="caster_sphere_link">
+    <visual>
+      <geometry>
+        <sphere radius="${caster_sphere_radius}"/>
+      </geometry>
+    </visual>
+    <collision>
+      <geometry>
+        <sphere radius="${caster_sphere_radius}"/>
+      </geometry>
+    </collision>
+    <inertial>
+      <mass value="${caster_sphere_mass}"/>
+      <inertia
+        ixx="${2 * caster_sphere_mass * caster_sphere_radius *
+               caster_sphere_radius / 5}"
+        ixy="0.0" ixz="0.0"
+        iyy="${2 * caster_sphere_mass * caster_sphere_radius *
+               caster_sphere_radius / 5}"
+        iyz="0.0"
+        izz="${2 * caster_sphere_mass * caster_sphere_radius *
+               caster_sphere_radius / 5}"/>
+    </inertial>
+  </link>
+  <!-- ========================================================= -->
   <!-- Left Wheel Joint                                            -->
   <!-- ========================================================= -->
@@ -119,5 +154,5 @@
     <child link="left_wheel_link"/>
     <!-- Wheel center -->
-    <origin xyz="0 ${s/2} ${wheel_radius/2}"
+    <origin xyz="0.1 ${s/2} ${wheel_radius/2}"
             rpy="0 0 0"/>
     <!-- Wheel rotates around Y -->
@@ -132,9 +167,14 @@
     <child link="right_wheel_link"/>
     <!-- Wheel center -->
-    <origin xyz="0 -${s/2} ${wheel_radius/2}"
+    <origin xyz="0.1 -${s/2} ${wheel_radius/2}"
             rpy="0 0 0"/>
     <!-- Wheel rotates around Y -->
     <axis xyz="0 1 0"/>
   </joint>
+  <joint name="caster_sphere_joint" type="fixed">
+    <parent link="base_link"/>
+    <child link="caster_sphere_link"/>
+    <origin xyz="-${caster_sphere_x} 0 ${caster_sphere_z}" rpy="0 0 0"/>
+  </joint>
   <xacro:include filename="$(find diff_drive_robot)/urdf/gazebo.xacro"/>
 </robot>

Commit message: Moved the baselink frame to the origin of the robot so i can get a good tracking of pose

File: src/diff_drive_robot/urdf/diff_drive_robot.xacro (robot description, xacro)
@@ -19,5 +19,5 @@
   <xacro:property name="caster_sphere_mass" value="0.20"/>
   <xacro:property name="caster_sphere_x"
-                  value="0.22"/>
+                  value="0.32"/>
   <!-- Sphere bottom matches the drive wheels' contact height. -->
   <xacro:property name="caster_sphere_z"
@@ -32,5 +32,5 @@
     <visual>
       <!-- Put the bottom of the body at z = 0 -->
-      <origin xyz="0 0 ${body_height/2}" rpy="0 0 0"/>
+      <origin xyz="-0.1 0 ${body_height/2}" rpy="0 0 0"/>
       <geometry>
         <box size="${body_length} ${body_width} ${body_height}"/>
@@ -154,5 +154,5 @@
     <child link="left_wheel_link"/>
     <!-- Wheel center -->
-    <origin xyz="0.1 ${s/2} ${wheel_radius/2}"
+    <origin xyz="0 ${s/2} ${wheel_radius/2}"
             rpy="0 0 0"/>
     <!-- Wheel rotates around Y -->
@@ -167,5 +167,5 @@
     <child link="right_wheel_link"/>
     <!-- Wheel center -->
-    <origin xyz="0.1 -${s/2} ${wheel_radius/2}"
+    <origin xyz="0 -${s/2} ${wheel_radius/2}"
             rpy="0 0 0"/>
     <!-- Wheel rotates around Y -->

Commit message: Edited the readme file

File: src/diff_drive_robot/urdf/diff_drive_robot.xacro (robot description, xacro)
@@ -11,5 +11,5 @@
   <!-- Differential-drive geometry -->
   <!-- s = distance between left and right wheel centers -->
-  <xacro:property name="s" value="0.40"/>
+  <xacro:property name="s" value="0.4"/>
   <!-- Wheels -->
   <xacro:property name="wheel_radius" value="0.10"/>
@@ -38,5 +38,5 @@
     </visual>
     <collision>
-      <origin xyz="0 0 ${body_height/2}" rpy="0 0 0"/>
+      <origin xyz="-0.1 0 ${body_height/2}" rpy="0 0 0"/>
       <geometry>
         <box size="${body_length} ${body_width} ${body_height}"/>
@@ -44,5 +44,5 @@
     </collision>
     <inertial>
-      <origin xyz="0 0 ${body_height/2}" rpy="0 0 0"/>
+      <origin xyz="-0.1 0 ${body_height/2}" rpy="0 0 0"/>
       <mass value="${body_mass}"/>
       <!-- Box inertia -->

File: src/diff_drive_robot/urdf/gazebo.xacro (robot description, xacro)
@@ -9,15 +9,15 @@
   <gazebo reference="left_wheel_link">
     <material>Gazebo/Black</material>
-    <mu1>1.0</mu1>
-    <mu2>1.0</mu2>
-    <kp>1000000.0</kp>
-    <kd>100.0</kd>
+    <mu1>1.5</mu1>
+    <mu2>1.5</mu2>
+    <kp>100000</kp>
+    <kd>10</kd>
   </gazebo>
   <gazebo reference="right_wheel_link">
     <material>Gazebo/Black</material>
-    <mu1>1.0</mu1>
-    <mu2>1.0</mu2>
-    <kp>1000000.0</kp>
-    <kd>100.0</kd>
+    <mu1>1.5</mu1>
+    <mu2>1.5</mu2>
+    <kp>100000.0</kp>
+    <kd>10</kd>
   </gazebo>
   <gazebo reference="caster_sphere_link">
@@ -26,6 +26,6 @@
     <mu1>0.02</mu1>
     <mu2>0.02</mu2>
-    <kp>1000000.0</kp>
-    <kd>100.0</kd>
+    <kp>100000</kp>
+    <kd>100</kd>
   </gazebo>
   <!-- ========================================================= -->
@@ -43,5 +43,5 @@
       <!-- Maximum velocities -->
       <max_wheel_torque>10.0</max_wheel_torque>
-      <max_wheel_acceleration>10.0</max_wheel_acceleration>
+      <max_wheel_acceleration>100.0</max_wheel_acceleration>
       <!-- Topics -->
       <command_topic>cmd_vel</command_topic>
